File: wclock.sch (EAGLE design)
At the start: 39 parts, among them IC1 DS1305, IC2 7805T, J1 DCJ0202, Q1 32.768KHz

Commit message: added missing wire to schematic
Connections:
- new net N$26: R11.2, R12.1
Changed lines of the file:
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@@
+</segment>
+</net>
+<net name="N$26" class="0">
+<segment>
+<pinref part="R11" gate="G$1" pin="2"/>
+<pinref part="R12" gate="G$1" pin="1"/>
+<wire x1="261.62" y1="2.54" x2="259.08" y2="2.54" width="0.1524" layer="91"/>
 </segment>
 </net>
